File: old_files_backup_20250614/MHT1803_Amplifier_500W_backup.kicad_sch (KiCad schematic)
At the start: 62 parts, among them J1 POWER_12V, J2 SO239_INPUT, J3 SO239_OUTPUT, K1 THERMAL_RELAY, K2 G5V-2-12V, K3 G5V-2-12V, K4 G5V-2-12V, Q1 MHT1803, Q2 MHT1803, SW1 POWER, SW2 BAND_SELECT, T1 RF_Transformer_4to1, T2 RF_Transformer_4to1, U1 LM25122MY, U2 LM393, U3 Arduino_Nano, U4 LCD_20x4, U5 ACS712_30A, U6 DC_DC_Converter

Commit message: split schematics to smaller, separate files per section
Parts:
- removed R6: 2.2kohm, Resistor_SMD:R_0805_2012Metric, symbol Device:R
- C1, C7: value 1000uF -> 1000µF
- C8: value 2200uF -> 2200µF
- FB1, FB2: value 1000ohm@100MHz -> 1000Ω@100MHz
- L3: value 100uH -> 100µH
- L4: value 2.2uH -> 2.2µH
- L5: value 1.0uH -> 1.0µH
- L6: value 0.47uH -> 0.47µH
- R1, R2: value 10ohm -> 10Ω
- R5: value 10kohm -> 10kΩ
- R6: renamed from U6; value DC_DC_Converter -> 2.2kΩ; footprint MHT1803_Amplifier_500W:DC_DC_Converter_Module -> Resistor_SMD:R_0805_2012Metric; symbol MHT1803_Amplifier_500W:DC_DC_Converter -> Device:R
- R7: value 0.01ohm -> 0.01Ω
- R8: value 1Mohm -> 1MΩ
- R9: value 50ohm -> 50Ω
- TH1: value 10kohm_NTC -> 10kΩ_NTC
Connections:
- net +50V: now also Q1.4 (Thermal), Q2.2 (S), Q2.4 (Thermal), R6.1, R6.2
Other:
- note added: "SECTION 5 - CONTROL AND MONITORING COMPLETED: 1. MICROCONTROLLER SYSTEM: - U3 (Arduino Nano): Main control processor - ATmega328P with 32KB flash, 2KB RAM - 16MHz crystal for precise timing - USB programming interface - Real-time monitoring and control algorithms 2. USER INTERFACE: - U4 (LCD 20x4): Alphanumeric display - SW1 (Power): Main power on/off switch - SW2 (Band Select): 12-position rotar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"
- note added: "SECTION 6: EMI/RFI FILTERING Components: - FB1, FB2: 1000Ω@100MHz ferrite beads for HF suppression - C9: 100nF bypass capacitor for mid-frequency filtering - C10: 10nF bypass capacitor for high-frequency filtering - C11: 1nF bypass capacitor for VHF/UHF filtering - L3: 100µH common mode choke for differential mode suppression - R8: 1MΩ discharge resistor for safety Filtering Performance: - Attenu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"
- note added: "SECTION 7: BAND SWITCHING/RELAY CONTROL Components: - K2, K3, K4: G5V-2 DPDT relays (12V coil, 2A contacts) - L4: 2.2µH inductor (160m/80m bands) - L5: 1.0µH inductor (40m/20m bands) - L6: 0.47µH inductor (15m/10m bands) - C12: 470pF capacitor (160m/80m bands) - C13: 220pF capacitor (40m/20m bands) - C14: 100pF capacitor (15m/10m bands) Band Selection Matrix: K2=0, K3=0, K4=0: 160m (L4+C12: 2.2µH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"
- note removed: "SECTION 5 - CONTROL AND MONITORING"
- note removed: "SECTION 6: EMI/RFI FILTERING"
- note removed: "SECTION 7: BAND SWITCHING/RELAY CONTROL"
